File: N64 U12 LDO Repair PCB.kicad_sch (KiCad schematic)
At the start: 5 parts, among them J1 Conn_01x05_Pin, U1 TLV78525PDBVR

Commit message: Revision 1: Fix pin pitch
Parts:
- J1: footprint Custom:CustomAdapter_TO-252-5 -> Custom:CustomAdapter_SharpPQ7VZ5; now not fitted
Changed lines of the file:
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@@
 		(on_board yes)
 		(in_pos_files yes)
-		(dnp no)
+		(dnp yes)
 		(fields_autoplaced yes)
 		(property "Reference" "J1"
@@
 			)
 		)
-		(property "Footprint" "Custom:CustomAdapter_TO-252-5"
+		(property "Footprint" "Custom:CustomAdapter_SharpPQ7VZ5"
 			(at 66.04 80.01 0)
 			(hide yes)
